File: ClawMachine.kicad_sch (KiCad schematic)
At the start: 86 parts, among them J1 Screw_Terminal_01x04, J10 Screw_Terminal_01x02, J11 Conn_01x02_Pin, J12 Screw_Terminal_01x02, J13 Conn_01x02_Pin, J14 Screw_Terminal_01x02, J15 Conn_01x02_Pin, J16 Screw_Terminal_01x02, J17 Conn_01x02_Pin, J18 Screw_Terminal_01x02, J19 Conn_01x02_Pin, J2 Screw_Terminal_01x04, J20 Screw_Terminal_01x02, J21 Conn_01x02_Pin, J22 Screw_Terminal_01x02, J23 Conn_01x02_Pin, J24 Screw_Terminal_01x02, J25 Conn_01x02_Pin, J26 Screw_Terminal_01x02, J27 Conn_01x02_Pin, J28 Conn_01x02_Pin, J29 Conn_01x02_Pin, J3 Screw_Terminal_01x02, J30 Conn_01x02_Pin, J31 Conn_01x02_Pin, J32 Conn_01x02_Pin, J4 Screw_Terminal_01x02, J5 Screw_Terminal_01x02, J6 Screw_Terminal_01x04, J7 Screw_Terminal_01x02, J8 Screw_Terminal_01x02, J9 Conn_01x02_Pin, Q1 AO3400A, Q2 AO3400A, Q3 AO3400A, Q4 AO3400A, SW1 SW_Push, SW10 SW_SPST, SW11 SW_Push, SW12 SW_SPST, SW13 SW_Push, SW14 SW_SPST, SW15 SW_Push, SW16 SW_SPST, SW17 SW_Push, SW18 SW_SPST, SW19 SW_Push, SW2 SW_SPST, SW20 SW_SPST, SW21 SW_Push, SW22 SW_Push, SW23 SW_Push, SW24 SW_Push, SW25 SW_Push, SW3 SW_Push, SW4 SW_SPST, SW5 SW_Push, SW6 SW_SPST, SW7 SW_Push, SW8 SW_SPST, SW9 SW_Push, U1 L298N, U2 L298N

Commit message: make more modular
Parts:
- removed J10, J12, J14, J16, J18, J20, J22, J24, J26, J8: Screw_Terminal_01x02, symbol Connector:Screw_Terminal_01x02
- removed J11, J13, J15, J17, J19, J21, J23, J25, J27, J28, J29, J30, J31, J32, J9: Conn_01x02_Pin, symbol Connector:Conn_01x02_Pin
- removed R10, R11, R12, R13, R14, R15, R16, R17, R18, R19, R5, R6, R7, R8, R9: R_US, symbol Device:R_US
- removed SW1, SW11, SW13, SW15, SW17, SW19, SW21, SW22, SW23, SW24, SW25, SW3, SW5, SW7, SW9: SW_Push, symbol Switch:SW_Push
- removed SW10, SW12, SW14, SW16, SW18, SW2, SW20, SW4, SW6, SW8: SW_SPST, symbol Switch:SW_SPST
Connections:
- net at A1.10 (MS1), A3.10 (MS1): no longer A4.D5
- net at A1.11 (MS2), A3.11 (MS2): no longer A4.D6
- net at A1.12 (MS3), A3.12 (MS3): no longer A4.D7
- net at A1.15 (STEP), A3.15 (STEP): no longer A4.D3 (D3_INT1)
- net at A1.16 (DIR), A3.16 (DIR): no longer A4.D4
- net at A1.9 (~{ENABLE}), A3.9 (~{ENABLE}): no longer A4.D2 (D2_INT0)
- net at A5.10 (MS1): no longer A4.D11
- net at A5.11 (MS2): no longer A4.D12
- net at A5.12 (MS3): no longer A4.D13
- net at A5.15 (STEP): no longer A4.D9
- net at A5.16 (DIR): no longer A4.D10
- net at A5.9 (~{ENABLE}): no longer A4.D8
- net at U1.5 (IN1): no longer A4.D22
- net at U1.7 (IN2): no longer A4.D23
- net at U1.6 (EnA): no longer A4.D24
- net at A4.D25: no longer U1.10 (IN3)
- net at A4.D26: no longer U1.12 (IN4)
- net at A4.D27: no longer U1.11 (EnB)
- net at A4.D28: no longer U2.5 (IN1)
- net at A4.D29: no longer U2.7 (IN2)
- net at A4.D30: no longer U2.6 (EnA)
- net at A4.D31: no longer U2.10 (IN3)
- net at A4.D32: no longer U2.12 (IN4)
- net at A4.D33: no longer U2.11 (EnB)
- new net control_stick_all/drop_input: A4.D24
- new net control_stick_all/east_input: A4.D23
- new net control_stick_all/north_input: A4.D12
- new net control_stick_all/south_input: A4.D13
- new net control_stick_all/west_input: A4.D22
- new net limit_switches_all/claw_close_limit: A4.D11
- new net limit_switches_all/claw_open_limit: A4.D10
- new net limit_switches_all/negative_x1_limit: A4.D3 (D3_INT1)
- new net limit_switches_all/negative_x2_limit: A4.D5
- new net limit_switches_all/negative_y_limit: A4.D7
- new net limit_switches_all/negative_z_limit: A4.D9
- new net limit_switches_all/positive_x1_limit: A4.D2 (D2_INT0)
- new net limit_switches_all/positive_x2_limit: A4.D4
- new net limit_switches_all/positive_y_limit: A4.D6
- new net limit_switches_all/positive_z_limit: A4.D8
Other:
- added sheet control_stick_all (control_stick_all.kicad_sch)
- added sheet limit_switches_all (limit_switches_all.kicad_sch)
- added sheet motor_driver_single (motor_driver.kicad_sch)
- added sheet stepper_driver_single (stepper_driver.kicad_sch)
- moved on the sheet: A1, A3, A5, J1, J2, J3, J4, J5, J6, J7, U1, U2

Commit message: add clk, drivers & pwr
Parts:
- removed A1, A3, A5: Pololu_Breakout_A4988, Module:Pololu_Breakout-16_15.2x20.3mm, symbol Driver_Motor:Pololu_Breakout_A4988
- removed J1, J2, J6: Screw_Terminal_01x04, symbol Connector:Screw_Terminal_01x04
- removed J3, J4, J5, J7: Screw_Terminal_01x02, symbol Connector:Screw_Terminal_01x02
- removed Q1, Q2, Q3, Q4: AO3400A, Package_TO_SOT_SMD:SOT-23, symbol Transistor_FET:AO3400A
- removed R1, R2, R3, R4: R_US, symbol Device:R_US
- removed U1, U2: L298N, Package_TO_SOT_THT:TO-220-15_P2.54x2.54mm_StaggerOdd_Lead4.58mm_Vertical, symbol Driver_Motor:L298N
Connections:
- net stepper_driver_all/y_stepper_driver_step: now reaches A4.D25
- net stepper_driver_all/y_stepper_driver_en: now reaches A4.D26
- net stepper_driver_all/y_stepper_driver_dir: now reaches A4.D27
- net stepper_driver_all/y_stepper_driver_ms1: now reaches A4.D28
- net stepper_driver_all/y_stepper_driver_ms2: now reaches A4.D29
- net stepper_driver_all/y_stepper_driver_ms3: now reaches A4.D30
- net stepper_driver_all/x_stepper_driver_step: now reaches A4.D31
- net stepper_driver_all/x_stepper_driver_en: now reaches A4.D32
- net stepper_driver_all/x_stepper_driver_dir: now reaches A4.D33
- net stepper_driver_all/x_stepper_driver_ms1: now reaches A4.D34
- net stepper_driver_all/x_stepper_driver_ms2: now reaches A4.D35
- net stepper_driver_all/x_stepper_driver_ms3: now reaches A4.D36
- net dc_driver_all/z_dc_in1: now reaches A4.D37
- net dc_driver_all/z_dc_in2: now reaches A4.D38
- net dc_driver_all/z_dc_in3: now reaches A4.D39
- net dc_driver_all/z_dc_in4: now reaches A4.D40
- net dc_driver_all/z_dc_ena: now reaches A4.D41
- net dc_driver_all/z_dc_enb: now reaches A4.D42
- net dc_driver_all/open_dc_in1: now reaches A4.D43
- net dc_driver_all/open_dc_in2: now reaches A4.D44
- net dc_driver_all/open_dc_in3: now reaches A4.D45
- net dc_driver_all/open_dc_in4: now reaches A4.D46
- net dc_driver_all/open_dc_ena: now reaches A4.D47
- net dc_driver_all/open_dc_enb: now reaches A4.D48
- net general_pwr_all/general_pwr_1: now reaches A4.D49
- net general_pwr_all/general_pwr_2: now reaches A4.D50 (D50_MISO)
- net general_pwr_all/general_pwr_3: now reaches A4.D51 (D51_MOSI)
- net general_pwr_all/general_pwr_4: now reaches A4.D52 (D52_SCK)
- net GND: now reaches A4.GND6 (GND)
- net countdown_clk/clk_scl: now reaches A4.SCL
- net countdown_clk/clk_sda: now reaches A4.SDA
- net +12V: now reaches A4.VIN
Other:
- removed sheet motor_driver_single
- removed sheet stepper_driver_single
- added sheet countdown_clk (countdown_clk.kicad_sch)
- added sheet dc_driver_all (dc_driver_all.kicad_sch)
- added sheet general_pwr_all (general_pwr_all.kicad_sch)
- added sheet stepper_driver_all (stepper_driver_all.kicad_sch)
