File: ClawMachine.kicad_pcb (KiCad board)
At the start: 2 copper layers, 10 parts, among them Q1 AO3400A, Q2 AO3400A, Q3 AO3400A, Q4 AO3400A, U1 L298N, U2 L298N

Commit message: add pcb? i think
Parts:
- removed A5: Pololu_Breakout_A4988, Module:Pololu_Breakout-16_15.2x20.3mm
- added A2: Pololu_Breakout_A4988, Module:Pololu_Breakout-16_15.2x20.3mm, F.Cu at (66.6, 125.0)
- added D1: LED, LED_THT:LED_D1.8mm_W1.8mm_H2.4mm_Horizontal_O1.27mm_Z1.6mm, F.Cu at (113.9, 147.4)
- added D2: LED, LED_THT:LED_D1.8mm_W1.8mm_H2.4mm_Horizontal_O1.27mm_Z1.6mm, F.Cu at (184.2, 143.6)
- added D3: LED, LED_THT:LED_D1.8mm_W1.8mm_H2.4mm_Horizontal_O1.27mm_Z1.6mm, F.Cu at (90.1, 147.0)
- added D4: LED, LED_THT:LED_D1.8mm_W1.8mm_H2.4mm_Horizontal_O1.27mm_Z1.6mm, F.Cu at (136.5, 147.4)
- added J1: Conn_01x02_Pin, Connector_PinHeader_2.54mm:PinHeader_1x02_P2.54mm_Vertical, F.Cu at (176.9, 134.9)
- added J10: Screw_Terminal_01x02, TerminalBlock:TerminalBlock_bornier-2_P5.08mm, F.Cu at (183.1, 107.0)
- added J11: Conn_01x02_Pin, Connector_PinHeader_2.54mm:PinHeader_1x02_P2.54mm_Vertical, F.Cu at (193.8, 104.8)
- added J12: Screw_Terminal_01x02, TerminalBlock:TerminalBlock_bornier-2_P5.08mm, F.Cu at (160.5, 107.0)
- added J13: Conn_01x02_Pin, Connector_PinHeader_2.54mm:PinHeader_1x02_P2.54mm_Vertical, F.Cu at (171.2, 104.8)
- added J14: Screw_Terminal_01x02, TerminalBlock:TerminalBlock_bornier-2_P5.08mm, F.Cu at (137.9, 128.6)
- added J15: Conn_01x02_Pin, Connector_PinHeader_2.54mm:PinHeader_1x02_P2.54mm_Vertical, F.Cu at (148.6, 126.4)
- added J16: Screw_Terminal_01x02, TerminalBlock:TerminalBlock_bornier-2_P5.08mm, F.Cu at (183.1, 85.5)
- added J17: Conn_01x02_Pin, Connector_PinHeader_2.54mm:PinHeader_1x02_P2.54mm_Vertical, F.Cu at (193.8, 83.3)
- added J18: Screw_Terminal_01x02, TerminalBlock:TerminalBlock_bornier-2_P5.08mm, F.Cu at (115.3, 85.5)
- added J19: Conn_01x02_Pin, Connector_PinHeader_2.54mm:PinHeader_1x02_P2.54mm_Vertical, F.Cu at (126.0, 83.3)
- added J2: Conn_01x02_Pin, Connector_PinHeader_2.54mm:PinHeader_1x02_P2.54mm_Vertical, F.Cu at (183.2, 66.4)
- added J20: Screw_Terminal_01x02, TerminalBlock:TerminalBlock_bornier-2_P5.08mm, F.Cu at (160.5, 85.5)
- added J21: Conn_01x02_Pin, Connector_PinHeader_2.54mm:PinHeader_1x02_P2.54mm_Vertical, F.Cu at (171.2, 83.3)
- added J22: Screw_Terminal_01x02, TerminalBlock:TerminalBlock_bornier-2_P5.08mm, F.Cu at (115.3, 107.0)
- added J23: Conn_01x02_Pin, Connector_PinHeader_2.54mm:PinHeader_1x02_P2.54mm_Vertical, F.Cu at (126.0, 104.8)
- added J24: Screw_Terminal_01x02, TerminalBlock:TerminalBlock_bornier-2_P5.08mm, F.Cu at (115.3, 128.6)
- added J25: Conn_01x02_Pin, Connector_PinHeader_2.54mm:PinHeader_1x02_P2.54mm_Vertical, F.Cu at (126.0, 126.4)
- added J26: Screw_Terminal_01x02, TerminalBlock:TerminalBlock_bornier-2_P5.08mm, F.Cu at (91.6, 129.7)
- added J27: Screw_Terminal_01x02, TerminalBlock:TerminalBlock_bornier-2_P5.08mm, F.Cu at (91.6, 138.7)
- added J28: Screw_Terminal_01x02, TerminalBlock:TerminalBlock_bornier-2_P5.08mm, F.Cu at (91.6, 97.5)
- added J29: Screw_Terminal_01x02, TerminalBlock:TerminalBlock_bornier-2_P5.08mm, F.Cu at (91.6, 106.6)
- added J3: Conn_01x02_Pin, Connector_PinHeader_2.54mm:PinHeader_1x02_P2.54mm_Vertical, F.Cu at (195.8, 66.4)
- added J30: Screw_Terminal_01x04, TerminalBlock:TerminalBlock_bornier-4_P5.08mm, F.Cu at (67.8, 118.4)
- added J31: Screw_Terminal_01x04, TerminalBlock:TerminalBlock_bornier-4_P5.08mm, F.Cu at (179.4, 27.2)
- added J32: Screw_Terminal_01x04, TerminalBlock:TerminalBlock_bornier-4_P5.08mm, F.Cu at (67.8, 85.5)
- added J4: Conn_01x02_Pin, Connector_PinHeader_2.54mm:PinHeader_1x02_P2.54mm_Vertical, F.Cu at (164.4, 134.9)
- added J5: Conn_01x02_Pin, Connector_PinHeader_2.54mm:PinHeader_1x02_P2.54mm_Vertical, F.Cu at (189.5, 134.9)
- added J6: Screw_Terminal_01x02, TerminalBlock:TerminalBlock_bornier-2_P5.08mm, F.Cu at (137.9, 107.0)
- added J7: Conn_01x02_Pin, Connector_PinHeader_2.54mm:PinHeader_1x02_P2.54mm_Vertical, F.Cu at (148.6, 104.8)
- added J8: Screw_Terminal_01x02, TerminalBlock:TerminalBlock_bornier-2_P5.08mm, F.Cu at (137.9, 85.5)
- added J9: Conn_01x02_Pin, Connector_PinHeader_2.54mm:PinHeader_1x02_P2.54mm_Vertical, F.Cu at (148.6, 83.3)
- added JP1: SolderJumper_3_Open, Jumper:SolderJumper-3_P1.3mm_Open_Pad1.0x1.5mm_NumberLabels, F.Cu at (114.9, 154.3)
- added JP2: SolderJumper_3_Open, Jumper:SolderJumper-3_P1.3mm_Open_Pad1.0x1.5mm_NumberLabels, F.Cu at (185.2, 150.5)
- added JP3: SolderJumper_3_Open, Jumper:SolderJumper-3_P1.3mm_Open_Pad1.0x1.5mm_NumberLabels, F.Cu at (91.2, 153.9)
- added JP4: SolderJumper_3_Open, Jumper:SolderJumper-3_P1.3mm_Open_Pad1.0x1.5mm_NumberLabels, F.Cu at (137.5, 154.3)
- added R1: R_US, Resistor_SMD:R_0805_2012Metric_Pad1.20x1.40mm_HandSolder, F.Cu at (172.2, 134.1)
- added R10: R_US, Resistor_SMD:R_0805_2012Metric_Pad1.20x1.40mm_HandSolder, F.Cu at (147.6, 142.1)
- added R11: R_US, Resistor_SMD:R_0805_2012Metric_Pad1.20x1.40mm_HandSolder, F.Cu at (192.8, 99.0)
- added R12: R_US, Resistor_SMD:R_0805_2012Metric_Pad1.20x1.40mm_HandSolder, F.Cu at (125.0, 99.0)
- added R13: R_US, Resistor_SMD:R_0805_2012Metric_Pad1.20x1.40mm_HandSolder, F.Cu at (170.2, 99.0)
- added R14: R_US, Resistor_SMD:R_0805_2012Metric_Pad1.20x1.40mm_HandSolder, F.Cu at (125.0, 120.6)
- added R15: R_US, Resistor_SMD:R_0805_2012Metric_Pad1.20x1.40mm_HandSolder, F.Cu at (125.0, 142.1)
- added R16: R, Resistor_SMD:R_0805_2012Metric_Pad1.20x1.40mm_HandSolder, F.Cu at (120.5, 147.1)
- added R17: R, Resistor_SMD:R_0805_2012Metric_Pad1.20x1.40mm_HandSolder, F.Cu at (120.5, 150.0)
- added R18: R, Resistor_SMD:R_0805_2012Metric_Pad1.20x1.40mm_HandSolder, F.Cu at (190.8, 143.3)
- added R19: R, Resistor_SMD:R_0805_2012Metric_Pad1.20x1.40mm_HandSolder, F.Cu at (190.8, 146.2)
- added R2: R_US, Resistor_SMD:R_0805_2012Metric_Pad1.20x1.40mm_HandSolder, F.Cu at (178.5, 65.6)
- added R20: R, Resistor_SMD:R_0805_2012Metric_Pad1.20x1.40mm_HandSolder, F.Cu at (96.8, 146.7)
- added R21: R, Resistor_SMD:R_0805_2012Metric_Pad1.20x1.40mm_HandSolder, F.Cu at (96.8, 149.7)
- added R22: R, Resistor_SMD:R_0805_2012Metric_Pad1.20x1.40mm_HandSolder, F.Cu at (143.1, 147.1)
- added R23: R, Resistor_SMD:R_0805_2012Metric_Pad1.20x1.40mm_HandSolder, F.Cu at (143.1, 150.0)
- added R3: R_US, Resistor_SMD:R_0805_2012Metric_Pad1.20x1.40mm_HandSolder, F.Cu at (191.1, 65.6)
- added R4: R_US, Resistor_SMD:R_0805_2012Metric_Pad1.20x1.40mm_HandSolder, F.Cu at (159.7, 134.1)
- added R5: R_US, Resistor_SMD:R_0805_2012Metric_Pad1.20x1.40mm_HandSolder, F.Cu at (184.8, 134.1)
- added R6: R_US, Resistor_SMD:R_0805_2012Metric_Pad1.20x1.40mm_HandSolder, F.Cu at (147.6, 120.6)
- added R7: R_US, Resistor_SMD:R_0805_2012Metric_Pad1.20x1.40mm_HandSolder, F.Cu at (147.6, 99.0)
- added R8: R_US, Resistor_SMD:R_0805_2012Metric_Pad1.20x1.40mm_HandSolder, F.Cu at (192.8, 120.6)
- added R9: R_US, Resistor_SMD:R_0805_2012Metric_Pad1.20x1.40mm_HandSolder, F.Cu at (170.2, 120.6)
- added SW1: SW_Push, Button_Switch_THT:SW_PUSH_6mm, F.Cu at (171.9, 126.1)
- added SW10: SW_Push, Button_Switch_THT:SW_PUSH_6mm, F.Cu at (181.9, 113.6)
- added SW11: SW_SPST, Button_Switch_SMD:SW_SPST_EVQP0, F.Cu at (195.5, 115.3)
- added SW12: SW_Push, Button_Switch_THT:SW_PUSH_6mm, F.Cu at (159.3, 113.6)
- added SW13: SW_SPST, Button_Switch_SMD:SW_SPST_EVQP0, F.Cu at (172.9, 115.3)
- added SW14: SW_Push, Button_Switch_THT:SW_PUSH_6mm, F.Cu at (136.7, 135.1)
- added SW15: SW_SPST, Button_Switch_SMD:SW_SPST_EVQP0, F.Cu at (150.3, 136.9)
- added SW16: SW_Push, Button_Switch_THT:SW_PUSH_6mm, F.Cu at (181.9, 92.0)
- added SW17: SW_SPST, Button_Switch_SMD:SW_SPST_EVQP0, F.Cu at (195.5, 93.8)
- added SW18: SW_Push, Button_Switch_THT:SW_PUSH_6mm, F.Cu at (114.1, 92.0)
- added SW19: SW_SPST, Button_Switch_SMD:SW_SPST_EVQP0, F.Cu at (127.7, 93.8)
- added SW2: SW_Push, Button_Switch_THT:SW_PUSH_6mm, F.Cu at (178.2, 57.6)
- added SW20: SW_Push, Button_Switch_THT:SW_PUSH_6mm, F.Cu at (159.3, 92.0)
- added SW21: SW_SPST, Button_Switch_SMD:SW_SPST_EVQP0, F.Cu at (172.9, 93.8)
- added SW22: SW_Push, Button_Switch_THT:SW_PUSH_6mm, F.Cu at (114.1, 113.6)
- added SW23: SW_SPST, Button_Switch_SMD:SW_SPST_EVQP0, F.Cu at (127.7, 115.3)
- added SW24: SW_Push, Button_Switch_THT:SW_PUSH_6mm, F.Cu at (114.1, 135.1)
- added SW25: SW_SPST, Button_Switch_SMD:SW_SPST_EVQP0, F.Cu at (127.7, 136.9)
- added SW3: SW_Push, Button_Switch_THT:SW_PUSH_6mm, F.Cu at (190.7, 57.6)
- added SW4: SW_Push, Button_Switch_THT:SW_PUSH_6mm, F.Cu at (159.3, 126.1)
- added SW5: SW_Push, Button_Switch_THT:SW_PUSH_6mm, F.Cu at (184.4, 126.1)
- added SW6: SW_Push, Button_Switch_THT:SW_PUSH_6mm, F.Cu at (136.7, 113.6)
- added SW7: SW_SPST, Button_Switch_SMD:SW_SPST_EVQP0, F.Cu at (150.3, 115.3)
- added SW8: SW_Push, Button_Switch_THT:SW_PUSH_6mm, F.Cu at (136.7, 92.0)
- added SW9: SW_SPST, Button_Switch_SMD:SW_SPST_EVQP0, F.Cu at (150.3, 93.8)
- A1: value Pololu_Breakout_A4988 -> Arduino_Mega2560_R3_Shield; footprint Module:Pololu_Breakout-16_15.2x20.3mm -> PCM_arduino-library:Arduino_Mega2560_R3_Shield
- A4: value Arduino_Mega2560_R3_Shield -> Pololu_Breakout_A4988; footprint PCM_arduino-library:Arduino_Mega2560_R3_Shield -> Module:Pololu_Breakout-16_15.2x20.3mm
- moved A3 126.0 mm to (178.2, 33.7)
- moved Q2 101.5 mm to (190.9, 149.9)
- moved Q1 76.5 mm to (120.6, 153.7)
- moved Q3 69.7 mm to (96.8, 153.4)
- moved Q4 68.8 mm to (143.2, 153.7)
- moved U1 38.1 mm to (90.3, 123.4)
- moved A1 28.6 mm to (71.8, 77.5)
- moved A4 26.0 mm to (66.6, 92.0)
- moved U2 6.97 mm to (90.3, 91.3)
Connections:
- A3 pad 1: Net-(U1-GND) -> (no net)
- A3 pad 10: Net-(A1-MS1) -> (no net)
- A3 pad 11: Net-(A1-MS2) -> (no net)
- A3 pad 12: Net-(A1-MS3) -> (no net)
- A3 pad 15: Net-(A1-STEP) -> (no net)
- A3 pad 16: Net-(A1-DIR) -> (no net)
- A3 pad 2: Net-(A1-VDD) -> (no net)
- A3 pad 7: Net-(U1-GND) -> (no net)
- A3 pad 8: Net-(A1-VMOT) -> (no net)
- A3 pad 9: Net-(A1-~{ENABLE}) -> (no net)
- Q1 pad 2: unconnected-(Q1-S-Pad2) -> (no net)
- Q1 pad 3: unconnected-(Q1-D-Pad3) -> (no net)
- Q2 pad 2: unconnected-(Q2-S-Pad2) -> (no net)
- Q2 pad 3: unconnected-(Q2-D-Pad3) -> (no net)
- Q3 pad 2: unconnected-(Q3-S-Pad2) -> (no net)
- Q3 pad 3: unconnected-(Q3-D-Pad3) -> (no net)
- Q4 pad 2: unconnected-(Q4-S-Pad2) -> (no net)
- Q4 pad 3: unconnected-(Q4-D-Pad3) -> (no net)
- U1 pad 1: Net-(U1-GND) -> (no net)
- U1 pad 10: Net-(U1-IN3) -> (no net)
- U1 pad 11: Net-(U1-EnB) -> (no net)
- U1 pad 12: Net-(U1-IN4) -> (no net)
- U1 pad 13: Net-(J4-Pin_1) -> (no net)
- U1 pad 14: Net-(J4-Pin_2) -> (no net)
- U1 pad 15: Net-(U1-GND) -> (no net)
- U1 pad 2: Net-(J3-Pin_1) -> (no net)
- U1 pad 3: Net-(J3-Pin_2) -> (no net)
- U1 pad 4: Net-(A1-VMOT) -> (no net)
- U1 pad 5: Net-(U1-IN1) -> (no net)
- U1 pad 6: Net-(U1-EnA) -> (no net)
- U1 pad 7: Net-(U1-IN2) -> (no net)
- U1 pad 8: Net-(U1-GND) -> (no net)
- U1 pad 9: Net-(A1-VDD) -> (no net)
- U2 pad 1: Net-(U1-GND) -> (no net)
- U2 pad 10: Net-(U2-IN3) -> (no net)
- U2 pad 11: Net-(U2-EnB) -> (no net)
- U2 pad 12: Net-(U2-IN4) -> (no net)
- U2 pad 13: Net-(J7-Pin_1) -> (no net)
- U2 pad 15: Net-(U1-GND) -> (no net)
- U2 pad 2: Net-(J5-Pin_1) -> (no net)
- U2 pad 4: Net-(A1-VMOT) -> (no net)
- U2 pad 5: Net-(U2-IN1) -> (no net)
- U2 pad 6: Net-(U2-EnA) -> (no net)
- U2 pad 7: Net-(U2-IN2) -> (no net)
- U2 pad 8: Net-(U1-GND) -> (no net)
- U2 pad 9: Net-(A1-VDD) -> (no net)
