File: claw_machine/control_stick.kicad_sch (KiCad schematic)
At the start: 3 parts, among them J32 Conn_01x02_Pin, SW25 SW_Push

Commit message: change folder stuff & update gen pwr
Parts:
- removed J32: Conn_01x02_Pin, symbol Connector:Conn_01x02_Pin
- removed R19: R_US, symbol Device:R_US
- removed SW25: SW_Push, symbol Switch:SW_Push
- added J5: Conn_01x02_Pin, Connector_PinHeader_2.54mm:PinHeader_1x02_P2.54mm_Vertical, symbol Connector:Conn_01x02_Pin
- added R5: R_US, Resistor_SMD:R_0805_2012Metric_Pad1.20x1.40mm_HandSolder, symbol Device:R_US
- added SW5: SW_Push, Button_Switch_THT:SW_PUSH_6mm, symbol Switch:SW_Push
Connections:
- net +5V: now also R5.2
- net GND: now also J5.1 (Pin_1), SW5.2
- net control_stick_input: now also J5.2 (Pin_2), R5.1, SW5.1
