File: claw_machine/dc_driver_all.kicad_sch (KiCad schematic)
At the start: 0 parts

Commit message: Rework schematic
Other:
- removed sheet dc_driver_single
- removed sheet dc_driver_single1
Changed lines of the file:
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@@
 (kicad_sch (version 20230121) (generator eeschema)
-  (paper "A4")
-  (wire (pts (xy 96.52 77.47) (xy 99.06 77.47))
-    (stroke (width 0) (type default))
-  )
-  (wire (pts (xy 96.52 82.55) (xy 99.06 82.55))
-    (stroke (width 0) (type default))
-  )
-  (wire (pts (xy 96.52 50.8) (xy 99.06 50.8))
-    (stroke (width 0) (type default))
-  )
-  (wire (pts (xy 96.52 62.23) (xy 99.06 62.23))
-    (stroke (width 0) (type default))
-  )
-  (wire (pts (xy 96.52 53.34) (xy 99.06 53.34))
-    (stroke (width 0) (type default))
-  )
-  (wire (pts (xy 96.52 88.9) (xy 99.06 88.9))
-    (stroke (width 0) (type default))
-  )
-  (wire (pts (xy 96.52 55.88) (xy 99.06 55.88))
-    (stroke (width 0) (type default))
-  )
-  (wire (pts (xy 96.52 64.77) (xy 99.06 64.77))
-    (stroke (width 0) (type default))
-  )
-  (wire (pts (xy 96.52 85.09) (xy 99.06 85.09))
-    (stroke (width 0) (type default))
-  )
-  (wire (pts (xy 96.52 91.44) (xy 99.06 91.44))
-    (stroke (width 0) (type default))
-  )
-  (wire (pts (xy 96.52 80.01) (xy 99.06 80.01))
-    (stroke (width 0) (type default))
-  )
-  (wire (pts (xy 96.52 58.42) (xy 99.06 58.42))
-    (stroke (width 0) (type default))
-  )
-  (hierarchical_label "open_dc_in1" (shape input) (at 96.52 77.47 180) (fields_autoplaced)
-    (effects (font (size 1.27 1.27)) (justify right))
-  )
-  (hierarchical_label "z_dc_in2" (shape input) (at 96.52 53.34 180) (fields_autoplaced)
-    (effects (font (size 1.27 1.27)) (justify right))
-  )
-  (hierarchical_label "z_dc_in3" (shape input) (at 96.52 55.88 180) (fields_autoplaced)
-    (effects (font (size 1.27 1.27)) (justify right))
-  )
-  (hierarchical_label "z_dc_in1" (shape input) (at 96.52 50.8 180) (fields_autoplaced)
-    (effects (font (size 1.27 1.27)) (justify right))
-  )
-  (hierarchical_label "open_dc_enb" (shape input) (at 96.52 91.44 180) (fields_autoplaced)
-    (effects (font (size 1.27 1.27)) (justify right))
-  )
-  (hierarchical_label "open_dc_in4" (shape input) (at 96.52 85.09 180) (fields_autoplaced)
-    (effects (font (size 1.27 1.27)) (justify right))
-  )
-  (hierarchical_label "z_dc_enb" (shape input) (at 96.52 64.77 180) (fields_autoplaced)
-    (effects (font (size 1.27 1.27)) (justify right))
-  )
-  (hierarchical_label "z_dc_ena" (shape input) (at 96.52 62.23 180) (fields_autoplaced)
-    (effects (font (size 1.27 1.27)) (justify right))
-  )
-  (hierarchical_label "open_dc_in3" (shape input) (at 96.52 82.55 180) (fields_autoplaced)
-    (effects (font (size 1.27 1.27)) (justify right))
-  )
-  (hierarchical_label "open_dc_ena" (shape input) (at 96.52 88.9 180) (fields_autoplaced)
-    (effects (font (size 1.27 1.27)) (justify right))
-  )
-  (hierarchical_label "z_dc_in4" (shape input) (at 96.52 58.42 180) (fields_autoplaced)
-    (effects (font (size 1.27 1.27)) (justify right))
-  )
-  (hierarchical_label "open_dc_in2" (shape input) (at 96.52 80.01 180) (fields_autoplaced)
-    (effects (font (size 1.27 1.27)) (justify right))
-  )
-  (sheet (at 99.06 48.26) (size 19.05 19.05)
-    (stroke (width 0.1524) (type solid))
-    (fill (color 0 0 0 0.0000))
-    (property "Sheetname" "dc_driver_single" (at 99.06 44.45 0)
-      (effects (font (size 1.27 1.27)) (justify left bottom))
-    )
-    (property "Sheetfile" "motor_driver.kicad_sch" (at 99.06 45.72 0)
-      (effects (font (size 1.27 1.27)) (justify left top))
-    )
-    (pin "IN1" input (at 99.06 50.8 180)
-      (effects (font (size 1.27 1.27)) (justify left))
-    )
-    (pin "IN2" input (at 99.06 53.34 180)
-      (effects (font (size 1.27 1.27)) (justify left))
-    )
-    (pin "EnA" input (at 99.06 62.23 180)
-      (effects (font (size 1.27 1.27)) (justify left))
-    )
-    (pin "EnB" input (at 99.06 64.77 180)
-      (effects (font (size 1.27 1.27)) (justify left))
-    )
-    (pin "IN4" input (at 99.06 58.42 180)
-      (effects (font (size 1.27 1.27)) (justify left))
-    )
-    (pin "IN3" input (at 99.06 55.88 180)
-      (effects (font (size 1.27 1.27)) (justify left))
-    )
-    (instances
-      (project "ClawMachine"
-        (path "/aafe1d38-cfbd-4a85-a256-fbe14cd8b9f5" (page "3"))
-        (path "/aafe1d38-cfbd-4a85-a256-fbe14cd8b9f5/a0269d26-c4d5-407d-802e-a17a1b6659b5" (page "3"))
-      )
-      (project "claw_machine"
-        (path "/2e48e9a4-e55f-4bd7-8086-6a8b9c5eabc1/c9c700bc-eabe-4388-8127-7a39929abe7a" (page "24"))
-      )
-    )
-  )
-  (sheet (at 99.06 74.93) (size 19.05 19.05)
-    (stroke (width 0.1524) (type solid))
-    (fill (color 0 0 0 0.0000))
-    (property "Sheetname" "dc_driver_single1" (at 99.06 71.12 0)
-      (effects (font (size 1.27 1.27)) (justify left bottom))
-    )
-    (property "Sheetfile" "motor_driver.kicad_sch" (at 99.06 72.39 0)
-      (effects (font (size 1.27 1.27)) (justify left top))
-    )
-    (pin "IN1" input (at 99.06 77.47 180)
-      (effects (font (size 1.27 1.27)) (justify left))
-    )
-    (pin "IN2" input (at 99.06 80.01 180)
-      (effects (font (size 1.27 1.27)) (justify left))
-    )
-    (pin "EnA" input (at 99.06 88.9 180)
-      (effects (font (size 1.27 1.27)) (justify left))
-    )
-    (pin "EnB" input (at 99.06 91.44 180)
-      (effects (font (size 1.27 1.27)) (justify left))
-    )
-    (pin "IN4" input (at 99.06 85.09 180)
-      (effects (font (size 1.27 1.27)) (justify left))
-    )
-    (pin "IN3" input (at 99.06 82.55 180)
-      (effects (font (size 1.27 1.27)) (justify left))
-    )
-    (instances
-      (project "ClawMachine"
-        (path "/aafe1d38-cfbd-4a85-a256-fbe14cd8b9f5" (page "3"))
-        (path "/aafe1d38-cfbd-4a85-a256-fbe14cd8b9f5/a0269d26-c4d5-407d-802e-a17a1b6659b5" (page "25"))
-      )
-      (project "claw_machine"
-        (path "/2e48e9a4-e55f-4bd7-8086-6a8b9c5eabc1/c9c700bc-eabe-4388-8127-7a39929abe7a" (page "23"))
-      )
-    )
-  )
+  (paper "USLetter")
 )
