File: claw_machine/claw_machine.kicad_pcb (KiCad board)
At the start: 2 copper layers, 98 parts, among them J1 Conn_01x02_Pin, J10 Screw_Terminal_01x02, J11 Conn_01x02_Pin, J12 Screw_Terminal_01x02, J13 Conn_01x02_Pin, J14 Screw_Terminal_01x02, J15 Conn_01x02_Pin, J16 Screw_Terminal_01x02, J17 Conn_01x02_Pin, J18 Screw_Terminal_01x02, J19 Conn_01x02_Pin, J2 Conn_01x02_Pin, J20 Screw_Terminal_01x02, J21 Conn_01x02_Pin, J22 Screw_Terminal_01x02, J23 Conn_01x02_Pin, J24 Screw_Terminal_01x02, J25 Conn_01x02_Pin, J26 Screw_Terminal_01x02, J27 Screw_Terminal_01x02, J28 Screw_Terminal_01x02, J29 Screw_Terminal_01x02, J3 Conn_01x02_Pin, J30 Screw_Terminal_01x04, J31 Screw_Terminal_01x04, J32 Screw_Terminal_01x04, J4 Conn_01x02_Pin, J5 Conn_01x02_Pin, J6 Screw_Terminal_01x02, J7 Conn_01x02_Pin, J8 Screw_Terminal_01x02, J9 Conn_01x02_Pin, Q1 AO3400A, Q2 AO3400A, Q3 AO3400A, Q4 AO3400A, SW1 SW_Push, SW10 SW_Push, SW11 SW_SPST, SW12 SW_Push, SW13 SW_SPST, SW14 SW_Push, SW15 SW_SPST, SW16 SW_Push, SW17 SW_SPST, SW18 SW_Push, SW19 SW_SPST, SW2 SW_Push, SW20 SW_Push, SW21 SW_SPST, SW22 SW_Push, SW23 SW_SPST, SW24 SW_Push, SW25 SW_SPST, SW3 SW_Push, SW4 SW_Push, SW5 SW_Push, SW6 SW_Push, SW7 SW_SPST, SW8 SW_Push, SW9 SW_SPST, U1 L298N, U2 L298N

Commit message: Start PCB work
Parts:
- removed A2, A3, A4: Pololu_Breakout_A4988, Module:Pololu_Breakout-16_15.2x20.3mm
- removed D1, D2, D3, D4: LED, LED_THT:LED_D1.8mm_W1.8mm_H2.4mm_Horizontal_O1.27mm_Z1.6mm
- removed J1, J11, J13, J15, J17, J19, J2, J21, J23, J25, J3, J4, J5, J7, J9: Conn_01x02_Pin, Connector_PinHeader_2.54mm:PinHeader_1x02_P2.54mm_Vertical
- removed J10, J12, J14, J16, J18, J20, J22, J24, J26, J27, J28, J29, J6, J8: Screw_Terminal_01x02, TerminalBlock:TerminalBlock_bornier-2_P5.08mm
- removed J30, J31, J32: Screw_Terminal_01x04, TerminalBlock:TerminalBlock_bornier-4_P5.08mm
- removed JP1, JP2, JP3, JP4: SolderJumper_3_Open, Jumper:SolderJumper-3_P1.3mm_Open_Pad1.0x1.5mm_NumberLabels
- removed Q1, Q2, Q3, Q4: AO3400A, Package_TO_SOT_SMD:SOT-23
- removed R1, R10, R11, R12, R13, R14, R15, R2, R3, R4, R5, R6, R7, R8, R9: R_US, Resistor_SMD:R_0805_2012Metric_Pad1.20x1.40mm_HandSolder
- removed R16, R17, R18, R19, R20, R21, R22, R23: R, Resistor_SMD:R_0805_2012Metric_Pad1.20x1.40mm_HandSolder
- removed SW1, SW10, SW12, SW14, SW16, SW18, SW2, SW20, SW22, SW24, SW3, SW4, SW5, SW6, SW8: SW_Push, Button_Switch_THT:SW_PUSH_6mm
- removed SW11, SW13, SW15, SW17, SW19, SW21, SW23, SW25, SW7, SW9: SW_SPST, Button_Switch_SMD:SW_SPST_EVQP0
- removed U1, U2: L298N, Package_TO_SOT_THT:TO-220-15_P2.54x2.54mm_StaggerOdd_Lead4.58mm_Vertical
- added A301: Pololu_Breakout_A4988, Module:Pololu_Breakout-16_15.2x20.3mm, F.Cu at (14.0, 165.1)
- added A401: Pololu_Breakout_A4988, Module:Pololu_Breakout-16_15.2x20.3mm, F.Cu at (-10.2, 165.1)
- added A501: Pololu_Breakout_A4988, Module:Pololu_Breakout-16_15.2x20.3mm, F.Cu at (-33.0, 165.1)
- added C1001: 10n, Capacitor_SMD:C_1206_3216Metric_Pad1.33x1.80mm_HandSolder, F.Cu at (232.8, 116.5)
- added C101: 100u, Capacitor_THT:CP_Radial_D10.0mm_P5.00mm_P7.50mm, F.Cu at (146.1, 44.5)
- added C102: 100u, Capacitor_THT:CP_Radial_D10.0mm_P5.00mm_P7.50mm, F.Cu at (146.7, 70.4)
- added C1101: 10n, Capacitor_SMD:C_1206_3216Metric_Pad1.33x1.80mm_HandSolder, F.Cu at (251.4, 77.3)
- added C1201: 10n, Capacitor_SMD:C_1206_3216Metric_Pad1.33x1.80mm_HandSolder, F.Cu at (251.4, 116.5)
- added C1301: 10n, Capacitor_SMD:C_1206_3216Metric_Pad1.33x1.80mm_HandSolder, F.Cu at (251.4, 97.0)
- added C1401: 10n, Capacitor_SMD:C_1206_3216Metric_Pad1.33x1.80mm_HandSolder, F.Cu at (232.8, 77.3)
- added C1501: 10n, Capacitor_SMD:C_1206_3216Metric_Pad1.33x1.80mm_HandSolder, F.Cu at (270.0, 77.3)
- added C201: 10n, Capacitor_SMD:C_1206_3216Metric_Pad1.33x1.80mm_HandSolder, F.Cu at (223.8, 56.7)
- added C202: 10n, Capacitor_SMD:C_1206_3216Metric_Pad1.33x1.80mm_HandSolder, F.Cu at (223.8, 60.1)
- added C203: 10n, Capacitor_SMD:C_1206_3216Metric_Pad1.33x1.80mm_HandSolder, F.Cu at (223.8, 63.4)
- added C204: 10n, Capacitor_SMD:C_1206_3216Metric_Pad1.33x1.80mm_HandSolder, F.Cu at (223.8, 66.8)
- added C801: 10n, Capacitor_SMD:C_1206_3216Metric_Pad1.33x1.80mm_HandSolder, F.Cu at (125.7, 160.0)
- added C901: 10n, Capacitor_SMD:C_1206_3216Metric_Pad1.33x1.80mm_HandSolder, F.Cu at (270.0, 97.0)
- added D1701: LED, LED_SMD:LED_1206_3216Metric_Pad1.42x1.75mm_HandSolder, F.Cu at (266.8, 130.4)
- added D1801: LED, LED_SMD:LED_1206_3216Metric_Pad1.42x1.75mm_HandSolder, F.Cu at (266.1, 51.0)
- added D1901: LED, LED_SMD:LED_1206_3216Metric_Pad1.42x1.75mm_HandSolder, F.Cu at (266.8, 148.4)
- added H101: MountingHole, MountingHole:MountingHole_4mm, F.Cu at (55.9, 25.4)
- added H102: MountingHole, MountingHole:MountingHole_4mm, F.Cu at (55.9, 132.1)
- added H103: MountingHole, MountingHole:MountingHole_4mm, F.Cu at (178.0, 25.4)
- added H104: MountingHole, MountingHole:MountingHole_4mm, F.Cu at (86.4, 167.6)
- added J1001: Conn_01x02, Connector_PinHeader_2.54mm:PinHeader_1x02_P2.54mm_Vertical, F.Cu at (225.2, 117.8)
- added J1002: Screw_Terminal_01x02, TerminalBlock:TerminalBlock_bornier-2_P5.08mm, F.Cu at (223.9, 124.2)
- added J101: Conn_01x04, Connector_PinHeader_2.54mm:PinHeader_1x04_P2.54mm_Vertical, F.Cu at (196.6, 59.0)
- added J102: Conn_01x04, Connector_PinHeader_2.54mm:PinHeader_1x04_P2.54mm_Vertical, F.Cu at (201.3, 59.0)
- added J103: Conn_01x04, Connector_PinHeader_2.54mm:PinHeader_1x04_P2.54mm_Vertical, F.Cu at (205.9, 59.0)
- added J1101: Conn_01x02, Connector_PinHeader_2.54mm:PinHeader_1x02_P2.54mm_Vertical, F.Cu at (243.8, 78.6)
- added J1102: Screw_Terminal_01x02, TerminalBlock:TerminalBlock_bornier-2_P5.08mm, F.Cu at (242.5, 85.0)
- added J1201: Conn_01x02, Connector_PinHeader_2.54mm:PinHeader_1x02_P2.54mm_Vertical, F.Cu at (243.8, 117.8)
- added J1202: Screw_Terminal_01x02, TerminalBlock:TerminalBlock_bornier-2_P5.08mm, F.Cu at (242.5, 124.2)
- added J12V_1: Screw_Terminal_01x02, TerminalBlock:TerminalBlock_bornier-2_P5.08mm, F.Cu at (141.0, 55.9)
- added J12V_2: Screw_Terminal_01x02, TerminalBlock:TerminalBlock_bornier-2_P5.08mm, F.Cu at (152.4, 55.9)
- added J1301: Conn_01x02, Connector_PinHeader_2.54mm:PinHeader_1x02_P2.54mm_Vertical, F.Cu at (243.8, 98.2)
- added J1302: Screw_Terminal_01x02, TerminalBlock:TerminalBlock_bornier-2_P5.08mm, F.Cu at (242.5, 104.6)
- added J1401: Conn_01x02, Connector_PinHeader_2.54mm:PinHeader_1x02_P2.54mm_Vertical, F.Cu at (225.2, 78.6)
- added J1402: Screw_Terminal_01x02, TerminalBlock:TerminalBlock_bornier-2_P5.08mm, F.Cu at (223.9, 85.0)
- added J1501: Conn_01x02, Connector_PinHeader_2.54mm:PinHeader_1x02_P2.54mm_Vertical, F.Cu at (262.3, 78.6)
- added J1502: Screw_Terminal_01x02, TerminalBlock:TerminalBlock_bornier-2_P5.08mm, F.Cu at (261.1, 85.0)
- added J1601: Screw_Terminal_01x02, TerminalBlock:TerminalBlock_bornier-2_P5.08mm, F.Cu at (260.4, 62.8)
- added J1602: Conn_01x02, Connector_PinHeader_2.54mm:PinHeader_1x02_P2.54mm_Vertical, F.Cu at (271.0, 60.6)
- added J1701: Screw_Terminal_01x02, TerminalBlock:TerminalBlock_bornier-2_P5.08mm, F.Cu at (261.1, 124.2)
- added J1702: Conn_01x02, Connector_PinHeader_2.54mm:PinHeader_1x02_P2.54mm_Vertical, F.Cu at (271.7, 122.0)
- added J1801: Screw_Terminal_01x02, TerminalBlock:TerminalBlock_bornier-2_P5.08mm, F.Cu at (260.4, 44.8)
- added J1802: Conn_01x02, Connector_PinHeader_2.54mm:PinHeader_1x02_P2.54mm_Vertical, F.Cu at (271.0, 42.6)
- added J1901: Screw_Terminal_01x02, TerminalBlock:TerminalBlock_bornier-2_P5.08mm, F.Cu at (261.1, 142.2)
- added J1902: Conn_01x02, Connector_PinHeader_2.54mm:PinHeader_1x02_P2.54mm_Vertical, F.Cu at (271.7, 140.0)
- added J201: Conn_01x05, Connector_PinHeader_2.54mm:PinHeader_1x05_P2.54mm_Vertical, F.Cu at (223.1, 42.6)
- added J301: Screw_Terminal_01x04, TerminalBlock:TerminalBlock_bornier-4_P5.08mm, F.Cu at (11.4, 190.5)
- added J401: Screw_Terminal_01x04, TerminalBlock:TerminalBlock_bornier-4_P5.08mm, F.Cu at (-11.4, 190.5)
- added J501: Screw_Terminal_01x04, TerminalBlock:TerminalBlock_bornier-4_P5.08mm, F.Cu at (-34.3, 190.5)
- added J5V_1: Screw_Terminal_01x02, TerminalBlock:TerminalBlock_bornier-2_P5.08mm, F.Cu at (140.3, 80.5)
- added J5V_2: Screw_Terminal_01x02, TerminalBlock:TerminalBlock_bornier-2_P5.08mm, F.Cu at (152.3, 80.5)
- added J601: Screw_Terminal_01x02, TerminalBlock:TerminalBlock_bornier-2_P5.08mm, F.Cu at (200.2, 97.0)
- added J602: Screw_Terminal_01x02, TerminalBlock:TerminalBlock_bornier-2_P5.08mm, F.Cu at (200.2, 106.1)
- added J701: Screw_Terminal_01x02, TerminalBlock:TerminalBlock_bornier-2_P5.08mm, F.Cu at (200.2, 129.2)
- added J702: Screw_Terminal_01x02, TerminalBlock:TerminalBlock_bornier-2_P5.08mm, F.Cu at (200.2, 138.2)
- added J801: Conn_01x02, Connector_PinHeader_2.54mm:PinHeader_1x02_P2.54mm_Vertical, F.Cu at (118.1, 161.3)
- added J802: Screw_Terminal_01x02, TerminalBlock:TerminalBlock_bornier-2_P5.08mm, F.Cu at (116.8, 167.6)
- added J901: Conn_01x02, Connector_PinHeader_2.54mm:PinHeader_1x02_P2.54mm_Vertical, F.Cu at (262.3, 98.2)
- added J902: Screw_Terminal_01x02, TerminalBlock:TerminalBlock_bornier-2_P5.08mm, F.Cu at (261.1, 104.6)
- added JP1601: SolderJumper_3_Open, Jumper:SolderJumper-3_P1.3mm_Open_Pad1.0x1.5mm_NumberLabels, F.Cu at (265.9, 72.5)
- added JP1701: SolderJumper_3_Open, Jumper:SolderJumper-3_P1.3mm_Open_Pad1.0x1.5mm_NumberLabels, F.Cu at (266.6, 133.9)
- added JP1801: SolderJumper_3_Open, Jumper:SolderJumper-3_P1.3mm_Open_Pad1.0x1.5mm_NumberLabels, F.Cu at (265.9, 54.5)
- added JP1901: SolderJumper_3_Open, Jumper:SolderJumper-3_P1.3mm_Open_Pad1.0x1.5mm_NumberLabels, F.Cu at (266.6, 151.8)
- added LED1601: LED, LED_SMD:LED_1206_3216Metric_Pad1.42x1.75mm_HandSolder, F.Cu at (266.1, 69.0)
- added LED_12V_101: LED, LED_SMD:LED_1206_3216Metric_Pad1.42x1.75mm_HandSolder, F.Cu at (203.3, 41.9)
- added LED_5V_101: LED, LED_SMD:LED_1206_3216Metric_Pad1.42x1.75mm_HandSolder, F.Cu at (203.3, 45.3)
- added LED_OB_101: LED, LED_SMD:LED_1206_3216Metric_Pad1.42x1.75mm_HandSolder, F.Cu at (203.3, 48.7)
- added Q1601: AO3400A, Package_TO_SOT_SMD:SOT-23, F.Cu at (271.5, 69.5)
- added Q1701: AO3400A, Package_TO_SOT_SMD:SOT-23, F.Cu at (272.2, 130.9)
- added Q1801: AO3400A, Package_TO_SOT_SMD:SOT-23, F.Cu at (271.5, 51.5)
- added Q1901: AO3400A, Package_TO_SOT_SMD:SOT-23, F.Cu at (272.2, 148.9)
- added R1001: 10k, Resistor_SMD:R_1206_3216Metric_Pad1.30x1.75mm_HandSolder, F.Cu at (176.2, 112.8)
- added R101: 3k3, Resistor_SMD:R_1206_3216Metric_Pad1.30x1.75mm_HandSolder, F.Cu at (197.3, 41.9)
- added R102: 3k3, Resistor_SMD:R_1206_3216Metric_Pad1.30x1.75mm_HandSolder, F.Cu at (197.3, 45.2)
- added R103: 2k2, Resistor_SMD:R_1206_3216Metric_Pad1.30x1.75mm_HandSolder, F.Cu at (197.3, 48.5)
- added R104: 2k2, Resistor_SMD:R_1206_3216Metric_Pad1.30x1.75mm_HandSolder, F.Cu at (197.3, 51.8)
- added R105: 10k, Resistor_SMD:R_1206_3216Metric_Pad1.30x1.75mm_HandSolder, F.Cu at (197.3, 55.0)
- added R1101: 10k, Resistor_SMD:R_1206_3216Metric_Pad1.30x1.75mm_HandSolder, F.Cu at (168.3, 107.5)
- added R1201: 10k, Resistor_SMD:R_1206_3216Metric_Pad1.30x1.75mm_HandSolder, F.Cu at (176.2, 118.1)
- added R1301: 10k, Resistor_SMD:R_1206_3216Metric_Pad1.30x1.75mm_HandSolder, F.Cu at (168.3, 118.1)
- added R1401: 10k, Resistor_SMD:R_1206_3216Metric_Pad1.30x1.75mm_HandSolder, F.Cu at (160.3, 122.7)
- added R1501: 10k, Resistor_SMD:R_1206_3216Metric_Pad1.30x1.75mm_HandSolder, F.Cu at (176.2, 107.5)
- added R1601: 2k2, Resistor_SMD:R_1206_3216Metric_Pad1.30x1.75mm_HandSolder, F.Cu at (260.1, 68.9)
- added R1602: 10k, Resistor_SMD:R_1206_3216Metric_Pad1.30x1.75mm_HandSolder, F.Cu at (260.1, 72.2)
- added R1701: 2k2, Resistor_SMD:R_1206_3216Metric_Pad1.30x1.75mm_HandSolder, F.Cu at (260.8, 130.3)
- added R1702: 10k, Resistor_SMD:R_1206_3216Metric_Pad1.30x1.75mm_HandSolder, F.Cu at (260.8, 133.6)
- added R1801: 2k2, Resistor_SMD:R_1206_3216Metric_Pad1.30x1.75mm_HandSolder, F.Cu at (260.1, 50.9)
- added R1802: 10k, Resistor_SMD:R_1206_3216Metric_Pad1.30x1.75mm_HandSolder, F.Cu at (260.1, 54.2)
- added R1901: 2k2, Resistor_SMD:R_1206_3216Metric_Pad1.30x1.75mm_HandSolder, F.Cu at (260.8, 148.3)
- added R1902: 10k, Resistor_SMD:R_1206_3216Metric_Pad1.30x1.75mm_HandSolder, F.Cu at (260.8, 151.6)
- added R201: 10k, Resistor_SMD:R_1206_3216Metric_Pad1.30x1.75mm_HandSolder, F.Cu at (160.3, 107.5)
- added R202: 10k, Resistor_SMD:R_1206_3216Metric_Pad1.30x1.75mm_HandSolder, F.Cu at (160.3, 110.8)
- added R203: 10k, Resistor_SMD:R_1206_3216Metric_Pad1.30x1.75mm_HandSolder, F.Cu at (160.3, 114.1)
- added R204: 10k, Resistor_SMD:R_1206_3216Metric_Pad1.30x1.75mm_HandSolder, F.Cu at (160.3, 117.4)
- added R801: 10k, Resistor_SMD:R_1206_3216Metric_Pad1.30x1.75mm_HandSolder, F.Cu at (125.7, 154.7)
- added R901: 10k, Resistor_SMD:R_1206_3216Metric_Pad1.30x1.75mm_HandSolder, F.Cu at (168.3, 123.4)
- added SW1001: SW_Push, Button_Switch_THT:SW_PUSH_6mm, F.Cu at (224.2, 113.5)
- added SW1101: SW_Push, Button_Switch_THT:SW_PUSH_6mm, F.Cu at (242.8, 74.2)
- added SW1201: SW_Push, Button_Switch_THT:SW_PUSH_6mm, F.Cu at (242.8, 113.5)
- added SW1301: SW_Push, Button_Switch_THT:SW_PUSH_6mm, F.Cu at (242.8, 93.8)
- added SW1401: SW_Push, Button_Switch_THT:SW_PUSH_6mm, F.Cu at (224.2, 74.2)
- added SW1501: SW_Push, Button_Switch_THT:SW_PUSH_6mm, F.Cu at (261.4, 74.2)
- added SW201: SW_Push, Button_Switch_THT:SW_PUSH_6mm, F.Cu at (212.3, 42.3)
- added SW202: SW_Push, Button_Switch_THT:SW_PUSH_6mm, F.Cu at (212.3, 50.8)
- added SW203: SW_Push, Button_Switch_THT:SW_PUSH_6mm, F.Cu at (212.3, 59.4)
- added SW204: SW_Push, Button_Switch_THT:SW_PUSH_6mm, F.Cu at (212.3, 67.9)
- added SW801: SW_Push, Button_Switch_THT:SW_PUSH_6mm, F.Cu at (117.1, 156.9)
- added SW901: SW_Push, Button_Switch_THT:SW_PUSH_6mm, F.Cu at (261.4, 93.8)
- added SW_RESET101: SW_Push, Button_Switch_THT:SW_PUSH_6mm, F.Cu at (196.3, 71.0)
- added U601: L298N, Package_TO_SOT_THT:TO-220-15_P2.54x2.54mm_StaggerOdd_Lead4.58mm_Vertical, F.Cu at (198.9, 90.8)
- added U701: L298N, Package_TO_SOT_THT:TO-220-15_P2.54x2.54mm_StaggerOdd_Lead4.58mm_Vertical, F.Cu at (198.9, 122.9)
- moved A101 54.9 mm to (62.2, 28.6), turned to -90 degrees
- renumbered A1 to A101
Connections:
- A101 pad 5V1: unconnected-(A1-5V-Pad5V1) -> +5V
- A101 pad 5V3: unconnected-(A1-5V-Pad5V3) -> +5V
- A101 pad 5V4: unconnected-(A1-5V-Pad5V4) -> +5V
- A101 pad A0: unconnected-(A1-PadA0) -> Net-(J103-Pin_1)
- A101 pad A1: unconnected-(A1-PadA1) -> Net-(J103-Pin_2)
- A101 pad A2: unconnected-(A1-PadA2) -> Net-(J103-Pin_3)
- A101 pad A3: unconnected-(A1-PadA3) -> Net-(J103-Pin_4)
- A101 pad D0: unconnected-(A1-D0/RX0-PadD0) -> Net-(A101-D0/RX0)
- A101 pad D1: unconnected-(A1-D1/TX0-PadD1) -> Net-(A101-D1/TX0)
- A101 pad D10: /limit_switches_all/claw_open_limit -> unconnected-(A101-PadD10)
- A101 pad D11: /limit_switches_all/claw_close_limit -> unconnected-(A101-PadD11)
- A101 pad D12: /control_stick_all/north_input -> unconnected-(A101-PadD12)
- A101 pad D13: /control_stick_all/south_input -> /ONBOARD_LED
- A101 pad D18: unconnected-(A1-D18/TX1-PadD18) -> Net-(A101-D18/TX1)
- A101 pad D19: unconnected-(A1-D19/RX1-PadD19) -> Net-(A101-D19/RX1)
- A101 pad D2: /limit_switches_all/positive_x1_limit -> /X1_LIMIT
- A101 pad D22: /control_stick_all/west_input -> /control_stick_all/NORTH_BTN
- A101 pad D23: /control_stick_all/east_input -> /control_stick_all/EAST_BTN
- A101 pad D24: /control_stick_all/drop_input -> /control_stick_all/SOUTH_BTN
- A101 pad D25: /stepper_driver_all/y_stepper_driver_step -> /control_stick_all/WEST_BTN
- A101 pad D26: /stepper_driver_all/y_stepper_driver_en -> /~{X1_EN}
- A101 pad D27: /stepper_driver_all/y_stepper_driver_dir -> /X1_STEP
- A101 pad D28: /stepper_driver_all/y_stepper_driver_ms1 -> /X1_DIR
- A101 pad D29: /stepper_driver_all/y_stepper_driver_ms2 -> /~{X2_EN}
- A101 pad D3: /limit_switches_all/negative_x1_limit -> /X2_LIMIT
- A101 pad D30: /stepper_driver_all/y_stepper_driver_ms3 -> /X2_STEP
- A101 pad D31: /stepper_driver_all/x_stepper_driver_step -> /X2_DIR
- A101 pad D32: /stepper_driver_all/x_stepper_driver_en -> /~{Y_EN}
- A101 pad D33: /stepper_driver_all/x_stepper_driver_dir -> /Y_STEP
- A101 pad D34: /stepper_driver_all/x_stepper_driver_ms1 -> /Y_DIR
- A101 pad D35: /stepper_driver_all/x_stepper_driver_ms2 -> /Z_DC_IN1
- A101 pad D36: /stepper_driver_all/x_stepper_driver_ms3 -> /Z_DC_IN2
- A101 pad D37: /dc_driver_all/z_dc_in1 -> /Z_DC_IN3
- A101 pad D38: /dc_driver_all/z_dc_in2 -> /Z_DC_IN4
- A101 pad D39: /dc_driver_all/z_dc_in3 -> /Z_DC_EN_A
- A101 pad D4: /limit_switches_all/positive_x2_limit -> /Y_LIMIT
- A101 pad D40: /dc_driver_all/z_dc_in4 -> /Z_DC_EN_B
- A101 pad D41: /dc_driver_all/z_dc_ena -> /CLAW_DC_IN1
- A101 pad D42: /dc_driver_all/z_dc_enb -> /CLAW_DC_IN2
- A101 pad D43: /dc_driver_all/open_dc_in1 -> /CLAW_DC_IN3
- A101 pad D44: /dc_driver_all/open_dc_in2 -> /CLAW_DC_IN4
- A101 pad D45: /dc_driver_all/open_dc_in3 -> /CLAW_DC_EN_A
- A101 pad D46: /dc_driver_all/open_dc_in4 -> /CLAW_DC_EN_B
- A101 pad D47: /dc_driver_all/open_dc_ena -> /GENERAL_PWR_EN_0
- A101 pad D48: /dc_driver_all/open_dc_enb -> /GENERAL_PWR_EN_1
- A101 pad D49: /general_pwr_all/general_pwr_1 -> /GENERAL_PWR_EN_2
- A101 pad D5: /limit_switches_all/negative_x2_limit -> /INPUT_BTN_1
- A101 pad D50: /general_pwr_all/general_pwr_2 -> /GENERAL_PWR_EN_3
- A101 pad D51: /general_pwr_all/general_pwr_3 -> unconnected-(A101-D51_MOSI-PadD51)
- A101 pad D52: /general_pwr_all/general_pwr_4 -> unconnected-(A101-D52_SCK-PadD52)
- A101 pad D6: /limit_switches_all/positive_y_limit -> /INPUT_BTN_2
- A101 pad D7: /limit_switches_all/negative_y_limit -> /INPUT_BTN_3
- A101 pad D8: /limit_switches_all/positive_z_limit -> /AUX_SW_1
- A101 pad D9: /limit_switches_all/negative_z_limit -> /AUX_SW_2
- A101 pad GND1: unconnected-(A1-GND-PadGND1) -> GND
- A101 pad GND2: unconnected-(A1-GND-PadGND2) -> GND
- A101 pad GND3: unconnected-(A1-GND-PadGND3) -> GND
- A101 pad GND5: unconnected-(A1-GND-PadGND5) -> GND
- A101 pad RST1: unconnected-(A1-RESET-PadRST1) -> Net-(A101-RESET)
- A101 pad SCL: /countdown_clk/clk_scl -> I2C_SCL
- A101 pad SDA: /countdown_clk/clk_sda -> I2C_SDA
Routing:
- net /Y_LIMIT: track 0.00 -> 55.4 mm
- net /INPUT_BTN_2: track 0.00 -> 55.4 mm
- net /INPUT_BTN_1: track 0.00 -> 55.4 mm
- net /AUX_SW_1: track 0.00 -> 55.4 mm
- net /INPUT_BTN_3: track 0.00 -> 55.4 mm
- net /AUX_SW_2: track 0.00 -> 55.4 mm
- net /X2_LIMIT: track 0.00 -> 55.4 mm
- net +5V: track 0.00 -> 33.7 mm, vias 0 -> 15
- net /X1_LIMIT: track 0.00 -> 27.3 mm
- added copper zone on B.Cu, net +5V
- added copper zone on F.Cu, net GND
Other:
- board outline added: 284.5 x 199.4 mm
- board text added: "X1_LIMIT"
- board text added: "X1_MOTOR"
- board text added: "X2_MOTOR"
- board text added: "Y_MOTOR"

Commit message: Do most of the PCB layout
Parts:
- J201: value Conn_01x05 -> Conn_02x05_Odd_Even; footprint Connector_PinHeader_2.54mm:PinHeader_1x05_P2.54mm_Vertical -> Connector_PinHeader_2.54mm:PinHeader_2x05_P2.54mm_Vertical
- moved SW901 184.8 mm to (82.8, 141.7)
- moved C901 184.8 mm to (91.4, 144.8)
- moved J901 184.8 mm to (83.8, 146.1)
- moved J902 184.8 mm to (82.5, 152.4)
- moved J103 148.3 mm to (59.1, 79.4)
- moved SW_RESET101 141.1 mm to (55.2, 67.3), turned to 90 degrees
- moved C1101 140.1 mm to (128.6, 144.8)
- moved J1101 140.1 mm to (120.9, 146.1)
- moved SW1101 140.1 mm to (120.0, 141.7)
- moved J1102 140.1 mm to (119.7, 152.4)
- moved C1001 126.8 mm to (109.2, 144.8)
- moved J1001 126.8 mm to (101.6, 146.1)
- moved SW1001 126.8 mm to (100.6, 141.7)
- moved J1002 126.8 mm to (100.3, 152.4)
- moved H104 122.9 mm to (208.3, 152.4)
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Connections:
- A101 pad D22: /control_stick_all/NORTH_BTN -> /control_stick/NORTH_BTN
- A101 pad D23: /control_stick_all/EAST_BTN -> /control_stick/EAST_BTN
- A101 pad D24: /control_stick_all/SOUTH_BTN -> /control_stick/SOUTH_BTN
- A101 pad D25: /control_stick_all/WEST_BTN -> /control_stick/WEST_BTN
- C201 pad 2: /control_stick_all/WEST_BTN -> /control_stick/WEST_BTN
- C202 pad 2: /control_stick_all/NORTH_BTN -> /control_stick/NORTH_BTN
- C203 pad 2: /control_stick_all/SOUTH_BTN -> /control_stick/SOUTH_BTN
- C204 pad 2: /control_stick_all/EAST_BTN -> /control_stick/EAST_BTN
- J201 pad 1: /control_stick_all/NORTH_BTN -> /control_stick/NORTH_BTN
- J201 pad 2: /control_stick_all/EAST_BTN -> /control_stick/NORTH_BTN
- J201 pad 3: /control_stick_all/SOUTH_BTN -> /control_stick/EAST_BTN
- J201 pad 4: /control_stick_all/WEST_BTN -> /control_stick/EAST_BTN
- J201 pad 5: +5V -> /control_stick/SOUTH_BTN
- R201 pad 1: /control_stick_all/WEST_BTN -> /control_stick/WEST_BTN
- R202 pad 1: /control_stick_all/NORTH_BTN -> /control_stick/NORTH_BTN
- R203 pad 1: /control_stick_all/SOUTH_BTN -> /control_stick/SOUTH_BTN
- R204 pad 1: /control_stick_all/EAST_BTN -> /control_stick/EAST_BTN
- SW201 pad 2: /control_stick_all/WEST_BTN -> /control_stick/WEST_BTN
- SW202 pad 2: /control_stick_all/NORTH_BTN -> /control_stick/NORTH_BTN
- SW203 pad 2: /control_stick_all/SOUTH_BTN -> /control_stick/SOUTH_BTN
- SW204 pad 2: /control_stick_all/EAST_BTN -> /control_stick/EAST_BTN
Routing:
- net /Y_LIMIT: track 55.4 -> 27.3 mm
- net /INPUT_BTN_1: track 55.4 -> 27.3 mm
- net /INPUT_BTN_2: track 55.4 -> 27.3 mm
- net /AUX_SW_1: track 55.4 -> 27.3 mm
- net /INPUT_BTN_3: track 55.4 -> 27.3 mm
- net /AUX_SW_2: track 55.4 -> 27.3 mm
- net /X2_LIMIT: track 55.4 -> 27.3 mm
- net +5V: track 33.7 -> 18.0 mm, vias 15 -> 8
Other:
- board size 284.5 x 199.4 mm -> 162.6 x 133.3 mm
- board text added: "5V"
- board text added: "AUX_1"
- board text added: "AUX_2"
- board text added: "BUTTON_1"
- board text added: "BUTTON_2"
- board text added: "BUTTON_3"
- board text added: "JOY STICK"
- board text added: "N S E W"
- board text added: "RST"
- board text added: "X2_LIMIT"
- board text added: "Y_LIMIT"

Commit message: Route all power traced and replicated sections
Parts:
- A101: moved to B.Cu
- JP1601, JP1701, JP1801, JP1901: footprint Jumper:SolderJumper-3_P1.3mm_Open_Pad1.0x1.5mm_NumberLabels -> Jumper:SolderJumper-3_P1.3mm_Open_RoundedPad1.0x1.5mm_NumberLabels
- Q1601, Q1701, Q1801, Q1901: footprint Package_TO_SOT_SMD:SOT-23 -> Library:SOT-23-MassivePads-HandSolder
- moved J501 254.5 mm to (162.6, 29.2)
- moved A501 235.8 mm to (175.2, 54.6), turned to 180 degrees
- moved J401 221.9 mm to (141.0, 29.2)
- moved A401 198.7 mm to (154.9, 54.6), turned to 180 degrees
- moved J301 194.1 mm to (119.4, 29.2)
- moved A301 162.7 mm to (133.3, 54.6), turned to 180 degrees
- moved J201 156.9 mm to (52.8, 116.1)
- moved Q1601 144.6 mm to (194.4, 79.4)
- moved LED1601 140.9 mm to (192.2, 74.9)
- moved R1601 140.5 mm to (186.4, 73.7), turned to 180 degrees
- moved J1602 140.3 mm to (199.4, 75.6), turned to 180 degrees
- moved R1602 138.7 mm to (188.6, 79.1), turned to -90 degrees
- moved JP1601 133.4 mm to (200.0, 81.3)
- moved R1901 133.0 mm to (186.4, 38.1), turned to 180 degrees
- moved D1901 132.1 mm to (192.2, 39.4)
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Routing:
- net +12V: track 0.00 -> 400.0 mm
- net Net-(A401-1B): track 0.00 -> 28.3 mm
- net Net-(A301-1B): track 0.00 -> 26.1 mm
- net Net-(A501-1B): track 0.00 -> 25.6 mm
- net Net-(A401-1A): track 0.00 -> 23.7 mm
- net Net-(J702-Pin_2): track 0.00 -> 22.5 mm
- net Net-(A301-1A): track 0.00 -> 21.5 mm
- net Net-(J601-Pin_1): track 0.00 -> 21.4 mm
- net Net-(J602-Pin_2): track 0.00 -> 21.4 mm
- net Net-(A501-1A): track 0.00 -> 20.9 mm
- net Net-(J701-Pin_1): track 0.00 -> 20.4 mm
- net Net-(A101-RESET): track 0.00 -> 18.0 mm
- net Net-(J1801-Pin_2): track 0.00 -> 17.6 mm
- net Net-(J1901-Pin_2): track 0.00 -> 17.6 mm
- net Net-(J1701-Pin_2): track 0.00 -> 17.6 mm
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Other:
- board size 162.6 x 133.3 mm -> 162.6 x 133.4 mm
- board text added: "+"
- board text added: "-"
- board text added: "0"
- board text added: "1"
- board text added: "1-2=5V 2-3=12V"
- board text added: "2"
- board text added: "3"
- board text added: "4"
- board text added: "CLAW MOTOR"
- board text added: "D0"
- board text added: "D1"
- board text added: "D18"
- board text added: "D19"
- board text added: "DNP"
- board text added: "Do Not Populate"
- board text added: "E"
- board text added: "N"
- board text added: "S"
- board text added: "W"
- board text added: "Z MOTOR"

Commit message: Autoroute and clean up manually
Routing:
- net /AUX_SW_2: track 27.3 -> 188.9 mm, vias 0 -> 1
- net /GENERAL_PWR_EN_3: track 8.72 -> 154.4 mm, vias 0 -> 2
- net /X1_STEP: track 0.00 -> 144.6 mm, vias 0 -> 2
- net /GENERAL_PWR_EN_2: track 8.72 -> 152.5 mm, vias 0 -> 3
- net /AUX_SW_1: track 27.3 -> 170.9 mm, vias 0 -> 1
- net /~{X1_EN}: track 0.00 -> 140.6 mm, vias 0 -> 1
- net /Z_DC_IN2: track 0.00 -> 137.0 mm, vias 0 -> 1
- net /X1_DIR: track 0.00 -> 135.3 mm, vias 0 -> 2
- net /~{X2_EN}: track 0.00 -> 132.4 mm
- net /INPUT_BTN_3: track 27.3 -> 158.9 mm, vias 0 -> 1
- net /GENERAL_PWR_EN_0: track 8.72 -> 139.1 mm, vias 0 -> 2
- net /control_stick/EAST_BTN: track 0.00 -> 130.3 mm, vias 0 -> 3
- net /GENERAL_PWR_EN_1: track 8.72 -> 137.8 mm, vias 0 -> 3
- net GND: track 0.00 -> 127.6 mm, vias 0 -> 12
- net /Z_DC_IN1: track 0.00 -> 127.4 mm, vias 0 -> 3
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
Commit message: Tweaks
Parts:
- H101, H102, H103, H104: footprint MountingHole:MountingHole_4mm -> MountingHole:MountingHole_4.3mm_M4_Pad_TopBottom
- J101: value Conn_01x04 -> ~; footprint Connector_PinHeader_2.54mm:PinHeader_1x04_P2.54mm_Vertical -> Connector_PinHeader_2.54mm:PinHeader_2x04_P2.54mm_Vertical
Connections:
- J101 pad 2: I2C_SDA -> +5V
- J101 pad 3: I2C_SCL -> I2C_SDA
- J101 pad 4: GND -> I2C_SDA
Routing:
- net I2C_SDA: track 28.2 -> 33.9 mm
- net I2C_SCL: track 27.4 -> 33.0 mm
- net /CLAW_DC_IN2: track 112.8 -> 115.4 mm
- net /~{X1_EN}: track 140.6 -> 142.0 mm
- net +12V: track 405.3 -> 406.0 mm
- net /Z_DC_EN_B: track 123.2 -> 123.9 mm
Other:
- board text added: "12V"
- board text added: "Arduino Mega goes here"
- board text added: "G"
- board text added: "GND"
- board text added: "I2C"
- board text added: "SCL"
- board text added: "SDA"
