File: claw_machine/claw_machine.kicad_pcb (KiCad board)
At the start: 2 copper layers, 162.6 x 133.4 mm, 116 parts, among them J1001 Conn_01x02, J1002 Screw_Terminal_01x02, J102 Conn_01x04, J103 Conn_01x04, J1101 Conn_01x02, J1102 Screw_Terminal_01x02, J1201 Conn_01x02, J1202 Screw_Terminal_01x02, J12V_1 Screw_Terminal_01x02, J12V_2 Screw_Terminal_01x02, J1301 Conn_01x02, J1302 Screw_Terminal_01x02, J1401 Conn_01x02, J1402 Screw_Terminal_01x02, J1501 Conn_01x02, J1502 Screw_Terminal_01x02, J1601 Screw_Terminal_01x02, J1602 Conn_01x02, J1701 Screw_Terminal_01x02, J1702 Conn_01x02, J1801 Screw_Terminal_01x02, J1802 Conn_01x02, J1901 Screw_Terminal_01x02, J1902 Conn_01x02, J201 Conn_02x05_Odd_Even, J301 Screw_Terminal_01x04, J401 Screw_Terminal_01x04, J501 Screw_Terminal_01x04, J5V_1 Screw_Terminal_01x02, J5V_2 Screw_Terminal_01x02, J601 Screw_Terminal_01x02, J602 Screw_Terminal_01x02, J701 Screw_Terminal_01x02, J702 Screw_Terminal_01x02, J801 Conn_01x02, J802 Screw_Terminal_01x02, J901 Conn_01x02, J902 Screw_Terminal_01x02, Q1601 AO3400A, Q1701 AO3400A, Q1801 AO3400A, Q1901 AO3400A, SW1001 SW_Push, SW1101 SW_Push, SW1201 SW_Push, SW1301 SW_Push, SW1401 SW_Push, SW1501 SW_Push, SW201 SW_Push, SW202 SW_Push, SW203 SW_Push, SW204 SW_Push, SW801 SW_Push, SW901 SW_Push, U601 L298N, U701 L298N

Commit message: Add names
Routing:
- net /INPUT_BTN_2: track 144.7 -> 143.7 mm
Other:
- board text added: "Emily Parker Jaxon Aleks Elyse Desly"
- board text added: "GNCTR 2024 Claw Game Toy Story Rev1"
- board text added: "GNCTR 2024 Claw Game Toy Story {dblquote}Bogg Story{dblquote}"
- board text added: "Rev1 2023-10-28"

Commit message: Finish, Gerbers
Parts:
- removed J601, J602: Screw_Terminal_01x02, TerminalBlock:TerminalBlock_bornier-2_P5.08mm
- removed U601: L298N, Package_TO_SOT_THT:TO-220-15_P2.54x2.54mm_StaggerOdd_Lead4.58mm_Vertical
- added J104: Conn_02x06_Odd_Even, Connector_PinHeader_2.54mm:PinHeader_2x06_P2.54mm_Vertical, F.Cu at (207.3, 110.9)
Connections:
- net Net-(J701-Pin_1) renamed /Z_OUT1
- net Net-(J701-Pin_2) renamed /Z_OUT2
- net Net-(J702-Pin_1) renamed /dc_driver_z/ OUT3
- net Net-(J702-Pin_2) renamed /dc_driver_z/ OUT4
- A101 pad D51: unconnected-(A101-D51_MOSI-PadD51) -> /Z_ENC_SIG_1
- A101 pad D52: unconnected-(A101-D52_SCK-PadD52) -> /Z_ENC_SIG_2
Routing:
- net /Z_ENC_SIG_2: track 0.00 -> 121.8 mm, vias 0 -> 1
- net /Z_ENC_SIG_1: track 0.00 -> 116.2 mm
- net /CLAW_DC_IN2: track 115.4 -> 0.00 mm, vias 2 -> 0
- net /CLAW_DC_IN1: track 111.7 -> 0.00 mm, vias 1 -> 0
- net /CLAW_DC_EN_A: track 110.5 -> 0.00 mm, vias 1 -> 0
- net /CLAW_DC_IN3: track 107.6 -> 0.00 mm, vias 1 -> 0
- net /CLAW_DC_IN4: track 104.4 -> 0.00 mm, vias 2 -> 0
- net /CLAW_DC_EN_B: track 102.5 -> 0.00 mm, vias 1 -> 0
- net +12V: track 406.0 -> 373.1 mm
- net /Z_OUT2: track 14.5 -> 43.5 mm
- net Net-(J602-Pin_2): track 21.7 -> 0.00 mm
- net Net-(J601-Pin_1): track 21.4 -> 0.00 mm
- net Net-(J602-Pin_1): track 15.5 -> 0.00 mm
- net Net-(J601-Pin_2): track 15.5 -> 0.00 mm
- net /Z_OUT1: track 20.4 -> 30.3 mm
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Other:
- board text added: "(MTR+/OUT1) Red[1] (ENC-) Black (SIG 1) Yellow (SIG 2) Green (ENC+) Blue (MTR-/OUT2) White"
- board text removed: "CLAW MOTOR"
