File: claw_machine/claw_machine.kicad_sch (KiCad schematic)
At the start: 1 part

Commit message: change folder stuff & update gen pwr
Parts:
- removed A4: Arduino_Mega2560_R3_Shield, PCM_arduino-library:Arduino_Mega2560_R3_Shield, symbol PCM_arduino-library:Arduino_Mega2560_R3_Shield
- added A1: Arduino_Mega2560_R3_Shield, PCM_arduino-library:Arduino_Mega2560_R3_Shield, symbol PCM_arduino-library:Arduino_Mega2560_R3_Shield
Connections:
- net +12V: now also A1.VIN
- net GND: now also A1.GND6 (GND)
- net control_stick_all/drop_input: now also A1.D24
- net control_stick_all/east_input: now also A1.D23
- net control_stick_all/north_input: now also A1.D12
- net control_stick_all/south_input: now also A1.D13
- net control_stick_all/west_input: now also A1.D22
- net countdown_clk/clk_scl: now also A1.SCL
- net countdown_clk/clk_sda: now also A1.SDA
- net dc_driver_all/open_dc_ena: now also A1.D47
- net dc_driver_all/open_dc_enb: now also A1.D48
- net dc_driver_all/open_dc_in1: now also A1.D43
- net dc_driver_all/open_dc_in2: now also A1.D44
- net dc_driver_all/open_dc_in3: now also A1.D45
- net dc_driver_all/open_dc_in4: now also A1.D46
- net dc_driver_all/z_dc_ena: now also A1.D41
- net dc_driver_all/z_dc_enb: now also A1.D42
- net dc_driver_all/z_dc_in1: now also A1.D37
- net dc_driver_all/z_dc_in2: now also A1.D38
- net dc_driver_all/z_dc_in3: now also A1.D39
- net dc_driver_all/z_dc_in4: now also A1.D40
- net general_pwr_all/general_pwr_1: now also A1.D49
- net general_pwr_all/general_pwr_2: now also A1.D50 (D50_MISO)
- net general_pwr_all/general_pwr_3: now also A1.D51 (D51_MOSI)
- net general_pwr_all/general_pwr_4: now also A1.D52 (D52_SCK)
- net limit_switches_all/claw_close_limit: now also A1.D11
- net limit_switches_all/claw_open_limit: now also A1.D10
- net limit_switches_all/negative_x1_limit: now also A1.D3 (D3_INT1)
- net limit_switches_all/negative_x2_limit: now also A1.D5
- net limit_switches_all/negative_y_limit: now also A1.D7
- net limit_switches_all/negative_z_limit: now also A1.D9
- net limit_switches_all/positive_x1_limit: now also A1.D2 (D2_INT0)
- net limit_switches_all/positive_x2_limit: now also A1.D4
- net limit_switches_all/positive_y_limit: now also A1.D6
- net limit_switches_all/positive_z_limit: now also A1.D8
- net stepper_driver_all/x_stepper_driver_dir: now also A1.D33
- net stepper_driver_all/x_stepper_driver_en: now also A1.D32
- net stepper_driver_all/x_stepper_driver_ms1: now also A1.D34
- net stepper_driver_all/x_stepper_driver_ms2: now also A1.D35
- net stepper_driver_all/x_stepper_driver_ms3: now also A1.D36
- net stepper_driver_all/x_stepper_driver_step: now also A1.D31
- net stepper_driver_all/y_stepper_driver_dir: now also A1.D27
- net stepper_driver_all/y_stepper_driver_en: now also A1.D26
- net stepper_driver_all/y_stepper_driver_ms1: now also A1.D28
- net stepper_driver_all/y_stepper_driver_ms2: now also A1.D29
- net stepper_driver_all/y_stepper_driver_ms3: now also A1.D30
- net stepper_driver_all/y_stepper_driver_step: now also A1.D25

Commit message: Rework schematic
Parts:
- added D1 (x3): LED, LED_THT:LED_D1.8mm_W1.8mm_H2.4mm_Horizontal_O1.27mm_Z1.6mm, symbol Device:LED
- added H101, H102, H103, H104: MountingHole, symbol Mechanical:MountingHole
- added J101, J102, J103: Conn_01x04, symbol Connector_Generic:Conn_01x04
- added J12V_1, J12V_2, J5V_1, J5V_2: Screw_Terminal_01x02, symbol Connector:Screw_Terminal_01x02
- added R101, R102: 3k3, symbol Device:R
- added R103, R104: 2k2, symbol Device:R
- added R105: 10k, symbol Device:R
- added SW4: SW_Push, Button_Switch_THT:SW_PUSH_6mm, symbol Switch:SW_Push
- renumbered A1 to A101
Connections:
- net +12V: now also J12V_1.1 (Pin_1), J12V_2.1 (Pin_1), R105.1
- net GND: now also A101.GND1 (GND), A101.GND2 (GND), A101.GND3 (GND), A101.GND5 (GND), D1.1 (K), D1.1 (K), D1.1 (K), J101.4 (Pin_4), J12V_1.2 (Pin_2), J12V_2.2 (Pin_2), J5V_1.2 (Pin_2), J5V_2.2 (Pin_2), SW4.1
- net +5V: now reaches A101.5V1 (5V)
- net +5V: now also A101.5V3 (5V), A101.5V4 (5V), J101.1 (Pin_1), J5V_1.1 (Pin_1), J5V_2.1 (Pin_1), R101.1, R102.1, R104.1
- net at A101.A0: now also J103.1 (Pin_1)
- net at A101.A1: now also J103.2 (Pin_2)
- net at A101.A2: now also J103.3 (Pin_3)
- net at A101.A3: now also J103.4 (Pin_4)
- net at A101.D0 (D0/RX0): now also J102.1 (Pin_1)
- net at A101.D1 (D1/TX0): now also J102.2 (Pin_2)
- net at A101.D18 (D18/TX1): now also J102.4 (Pin_4)
- net at A101.D19 (D19/RX1): now also J102.3 (Pin_3)
- net at A101.RST1 (RESET): now also SW4.2
- net control_stick_all/drop_input renamed control_stick_all/SOUTH_BTN
- net control_stick_all/east_input renamed control_stick_all/EAST_BTN
- net control_stick_all/north_input: no longer names the net of A101.D12
- net control_stick_all/south_input renamed ONBOARD_LED
- net ONBOARD_LED: now also R103.1
- net control_stick_all/west_input renamed control_stick_all/NORTH_BTN
- net countdown_clk/clk_scl renamed I2C_SCL
- net I2C_SCL: now also J101.3 (Pin_3), R101.2
- net countdown_clk/clk_sda renamed I2C_SDA
- net I2C_SDA: now also J101.2 (Pin_2), R102.2
- net dc_driver_all/open_dc_ena renamed GENERAL_PWR_EN_0
- net dc_driver_all/open_dc_enb renamed GENERAL_PWR_EN_1
- net dc_driver_all/open_dc_in1 renamed CLAW_DC_IN3
- net dc_driver_all/open_dc_in2 renamed CLAW_DC_IN4
- net dc_driver_all/open_dc_in3 renamed CLAW_DC_EN_A
- net dc_driver_all/open_dc_in4 renamed CLAW_DC_EN_B
- net dc_driver_all/z_dc_ena renamed CLAW_DC_IN1
- net dc_driver_all/z_dc_enb renamed CLAW_DC_IN2
- net dc_driver_all/z_dc_in1 renamed Z_DC_IN3
- net dc_driver_all/z_dc_in2 renamed Z_DC_IN4
- net dc_driver_all/z_dc_in3 renamed Z_DC_EN_A
- net dc_driver_all/z_dc_in4 renamed Z_DC_EN_B
- net general_pwr_all/general_pwr_1 renamed GENERAL_PWR_EN_2
- net general_pwr_all/general_pwr_2 renamed GENERAL_PWR_EN_3
- net general_pwr_all/general_pwr_3: no longer names the net of A101.D51 (D51_MOSI)
- net general_pwr_all/general_pwr_4: no longer names the net of A101.D52 (D52_SCK)
- net limit_switches_all/claw_close_limit: no longer names the net of A101.D11
- net limit_switches_all/claw_open_limit: no longer names the net of A101.D10
- net limit_switches_all/negative_x1_limit renamed X2_LIMIT
- net limit_switches_all/negative_x2_limit renamed INPUT_BTN_1
- net limit_switches_all/negative_y_limit renamed INPUT_BTN_3
- net limit_switches_all/negative_z_limit renamed AUX_SW_2
- net limit_switches_all/positive_x1_limit renamed X1_LIMIT
- net limit_switches_all/positive_x2_limit renamed Y_LIMIT
- net limit_switches_all/positive_y_limit renamed INPUT_BTN_2
- net limit_switches_all/positive_z_limit renamed AUX_SW_1
- net stepper_driver_all/x_stepper_driver_dir renamed Y_STEP
- net stepper_driver_all/x_stepper_driver_en renamed ~{Y_EN}
- net stepper_driver_all/x_stepper_driver_ms1 renamed Y_DIR
- net stepper_driver_all/x_stepper_driver_ms2 renamed Z_DC_IN1
- net stepper_driver_all/x_stepper_driver_ms3 renamed Z_DC_IN2
- net stepper_driver_all/x_stepper_driver_step renamed X2_DIR
- net stepper_driver_all/y_stepper_driver_dir renamed X1_STEP
- net stepper_driver_all/y_stepper_driver_en renamed ~{X1_EN}
- net stepper_driver_all/y_stepper_driver_ms1 renamed X1_DIR
- net stepper_driver_all/y_stepper_driver_ms2 renamed ~{X2_EN}
- net stepper_driver_all/y_stepper_driver_ms3 renamed X2_STEP
- net stepper_driver_all/y_stepper_driver_step renamed control_stick_all/WEST_BTN
- new net: D1.2 (A), R105.2
- new net: D1.2 (A), R103.2
- new net: D1.2 (A), R104.2
- no-connect marks 0 -> 27
Other:
- removed sheet countdown_clk
- removed sheet dc_driver_all
- removed sheet general_pwr_all
- removed sheet limit_switches_all
- removed sheet stepper_driver_all
- added sheet dc_driver_claw (motor_driver.kicad_sch)
- added sheet dc_driver_z (motor_driver.kicad_sch)
- added sheet general_pwr_single0 (general_pwr_single.kicad_sch)
- added sheet general_pwr_single1 (general_pwr_single.kicad_sch)
- added sheet general_pwr_single2 (general_pwr_single.kicad_sch)
- added sheet general_pwr_single3 (general_pwr_single.kicad_sch)
- added sheet stepper_driver_x1 (stepper_driver.kicad_sch)
- added sheet stepper_driver_x2 (stepper_driver.kicad_sch)
- added sheet stepper_driver_y (stepper_driver.kicad_sch)
- added sheet switch_aux_sw_1 (switch.kicad_sch)
- added sheet switch_aux_sw_2 (switch.kicad_sch)
- added sheet switch_input_btn_1 (switch.kicad_sch)
- added sheet switch_input_btn_2 (switch.kicad_sch)
- added sheet switch_input_btn_3 (switch.kicad_sch)
- added sheet switch_x1 (switch.kicad_sch)
- added sheet switch_x2 (switch.kicad_sch)
- added sheet switch_y (switch.kicad_sch)
- sheet control_stick_all ports: added EAST_BTN, NORTH_BTN, SOUTH_BTN, WEST_BTN; removed drop_input, east_input, north_input, south_input, west_input
- note added: "All Switches are Active High"
- note added: "DC Motor Drivers"
- note added: "Do Not Use 3V3"
- note added: "General Debug LED and Power LEDs"
- note added: "General Purpose MOSFET Drivers (LED Strips)"
- note added: "I2C for LCD"
- note added: "Microcontroller"
- note added: "Power Supply Mounting Holes"
- note added: "Stepper Drivers"
- note added: "Switches: Limit, Buttons, Aux"

Commit message: Assign footprints
Parts:
- H101, H102, H103, H104: footprint (none) -> MountingHole:MountingHole_4mm
- J101, J102, J103: footprint (none) -> Connector_PinHeader_2.54mm:PinHeader_1x04_P2.54mm_Vertical
- J12V_1, J12V_2, J5V_1, J5V_2: footprint (none) -> TerminalBlock:TerminalBlock_bornier-2_P5.08mm
- LED_12V_101, LED_5V_101, LED_OB_101: renamed from D1; footprint LED_THT:LED_D1.8mm_W1.8mm_H2.4mm_Horizontal_O1.27mm_Z1.6mm -> LED_SMD:LED_1206_3216Metric_Pad1.42x1.75mm_HandSolder
- R101, R102, R103, R104, R105: footprint (none) -> Resistor_SMD:R_1206_3216Metric_Pad1.30x1.75mm_HandSolder
Changed lines of the file:
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@@
       (effects (font (size 1.27 1.27)) (justify left) hide)
     )
-    (property "Footprint" "" (at 208.28 142.24 0)
+    (property "Footprint" "TerminalBlock:TerminalBlock_bornier-2_P5.08mm" (at 208.28 142.24 0)
       (effects (font (size 1.27 1.27)) hide)
     )
@@
       (effects (font (size 1.27 1.27)) (justify left) hide)
     )
-    (property "Footprint" "" (at 172.72 168.91 0)
+    (property "Footprint" "MountingHole:MountingHole_4mm" (at 172.72 168.91 0)
       (effects (font (size 1.27 1.27)) hide)
     )
@@
   (symbol (lib_id "Device:LED") (at 83.82 180.34 90) (unit 1)
     (in_bom yes) (on_board yes) (dnp no)
-    (property "Reference" "D1" (at 86.36 181.61 90)
+    (property "Reference" "LED_12V_101" (at 83.82 177.8 90)
       (effects (font (size 1.27 1.27)) (justify right))
     )
@@
       (effects (font (size 1.27 1.27)) (justify right) hide)
     )
-    (property "Footprint" "LED_THT:LED_D1.8mm_W1.8mm_H2.4mm_Horizontal_O1.27mm_Z1.6mm" (at 83.82 180.34 0)
+    (property "Footprint" "LED_SMD:LED_1206_3216Metric_Pad1.42x1.75mm_HandSolder" (at 83.82 180.34 0)
       (effects (font (size 1.27 1.27)) hide)
     )
@@
       (project "claw_machine"
         (path "/2e48e9a4-e55f-4bd7-8086-6a8b9c5eabc1"
-          (reference "LED_12V") (unit 1)
+          (reference "LED_12V_101") (unit 1)
         )
       )
@@
       (effects (font (size 1.27 1.27)) hide)
     )
-    (property "Footprint" "" (at 35.56 60.96 0)
+    (property "Footprint" "Connector_PinHeader_2.54mm:PinHeader_1x04_P2.54mm_Vertical" (at 35.56 60.96 0)
       (effects (font (size 1.27 1.27)) hide)
     )
@@
       (effects (font (size 1.27 1.27)) hide)
     )
-    (property "Footprint" "" (at 35.56 27.94 0)
+    (property "Footprint" "Connector_PinHeader_2.54mm:PinHeader_1x04_P2.54mm_Vertical" (at 35.56 27.94 0)
       (effects (font (size 1.27 1.27)) hide)
     )
@@
       (effects (font (size 1.27 1.27)) (justify left) hide)
     )
-    (property "Footprint" "" (at 162.56 163.83 0)
+    (property "Footprint" "MountingHole:MountingHole_4mm" (at 162.56 163.83 0)
       (effects (font (size 1.27 1.27)) hide)
     )
@@
       (effects (font (size 1.27 1.27)) (justify left))
     )
-    (property "Footprint" "" (at 64.008 170.18 90)
+    (property "Footprint" "Resistor_SMD:R_1206_3216Metric_Pad1.30x1.75mm_HandSolder" (at 64.008 170.18 90)
       (effects (font (size 1.27 1.27)) hide)
     )
@@
   (symbol (lib_id "Device:LED") (at 69.85 180.34 90) (unit 1)
     (in_bom yes) (on_board yes) (dnp no)
-    (property "Reference" "D1" (at 72.39 180.34 90)
+    (property "Reference" "LED_5V_101" (at 69.85 177.8 90)
       (effects (font (size 1.27 1.27)) (justify right))
     )
@@
       (effects (font (size 1.27 1.27)) (justify right) hide)
     )
-    (property "Footprint" "LED_THT:LED_D1.8mm_W1.8mm_H2.4mm_Horizontal_O1.27mm_Z1.6mm" (at 69.85 180.34 0)
+    (property "Footprint" "LED_SMD:LED_1206_3216Metric_Pad1.42x1.75mm_HandSolder" (at 69.85 180.34 0)
       (effects (font (size 1.27 1.27)) hide)
     )
@@
       (project "claw_machine"
         (path "/2e48e9a4-e55f-4bd7-8086-6a8b9c5eabc1"
-          (reference "LED_5V") (unit 1)
+          (reference "LED_5V_101") (unit 1)
         )
       )
@@
       (effects (font (size 1.27 1.27)) hide)
     )
-    (property "Footprint" "" (at 20.32 186.69 0)
+    (property "Footprint" "Connector_PinHeader_2.54mm:PinHeader_1x04_P2.54mm_Vertical" (at 20.32 186.69 0)
       (effects (font (size 1.27 1.27)) hide)
     )
@@
       (effects (font (size 1.27 1.27)) (justify left) hide)
     )
-    (property "Footprint" "" (at 162.56 168.91 0)
+    (property "Footprint" "MountingHole:MountingHole_4mm" (at 162.56 168.91 0)
       (effects (font (size 1.27 1.27)) hide)
     )
@@
       (effects (font (size 1.27 1.27)) (justify left) hide)
     )
-    (property "Footprint" "" (at 191.77 161.29 0)
+    (property "Footprint" "TerminalBlock:TerminalBlock_bornier-2_P5.08mm" (at 191.77 161.29 0)
       (effects (font (size 1.27 1.27)) hide)
     )
@@
       (effects (font (size 1.27 1.27)))
     )
-    (property "Footprint" "" (at 26.67 168.148 90)
+    (property "Footprint" "Resistor_SMD:R_1206_3216Metric_Pad1.30x1.75mm_HandSolder" (at 26.67 168.148 90)
       (effects (font (size 1.27 1.27)) hide)
     )
@@
       (effects (font (size 1.27 1.27)) (justify left) hide)
     )
-    (property "Footprint" "" (at 208.28 161.29 0)
+    (property "Footprint" "TerminalBlock:TerminalBlock_bornier-2_P5.08mm" (at 208.28 161.29 0)
       (effects (font (size 1.27 1.27)) hide)
     )
@@
       (effects (font (size 1.27 1.27)) (justify left))
     )
-    (property "Footprint" "" (at 68.072 170.18 90)
+    (property "Footprint" "Resistor_SMD:R_1206_3216Metric_Pad1.30x1.75mm_HandSolder" (at 68.072 170.18 90)
       (effects (font (size 1.27 1.27)) hide)
     )
@@
   (symbol (lib_id "Device:LED") (at 62.23 180.34 270) (mirror x) (unit 1)
     (in_bom yes) (on_board yes) (dnp no)
-    (property "Reference" "D1" (at 58.42 180.6575 90)
+    (property "Reference" "LED_OB_101" (at 60.96 177.8 90)
       (effects (font (size 1.27 1.27)) (justify right))
     )
@@
       (effects (font (size 1.27 1.27)) (justify right) hide)
     )
-    (property "Footprint" "LED_THT:LED_D1.8mm_W1.8mm_H2.4mm_Horizontal_O1.27mm_Z1.6mm" (at 62.23 180.34 0)
+    (property "Footprint" "LED_SMD:LED_1206_3216Metric_Pad1.42x1.75mm_HandSolder" (at 62.23 180.34 0)
       (effects (font (size 1.27 1.27)) hide)
     )
@@
       (project "claw_machine"
         (path "/2e48e9a4-e55f-4bd7-8086-6a8b9c5eabc1"
-          (reference "LED_OB") (unit 1)
+          (reference "LED_OB_101") (unit 1)
         )
       )
@@
       (effects (font (size 1.27 1.27)) (justify left))
     )
-    (property "Footprint" "" (at 82.042 170.18 90)
+    (property "Footprint" "Resistor_SMD:R_1206_3216Metric_Pad1.30x1.75mm_HandSolder" (at 82.042 170.18 90)
       (effects (font (size 1.27 1.27)) hide)
     )
@@
       (effects (font (size 1.27 1.27)) (justify left) hide)
     )
-    (property "Footprint" "" (at 191.77 142.24 0)
+    (property "Footprint" "TerminalBlock:TerminalBlock_bornier-2_P5.08mm" (at 191.77 142.24 0)
       (effects (font (size 1.27 1.27)) hide)
     )
@@
       (effects (font (size 1.27 1.27)) (justify left) hide)
     )
-    (property "Footprint" "" (at 172.72 163.83 0)
+    (property "Footprint" "MountingHole:MountingHole_4mm" (at 172.72 163.83 0)
       (effects (font (size 1.27 1.27)) hide)
     )
@@
       (effects (font (size 1.27 1.27)))
     )
-    (property "Footprint" "" (at 26.67 167.132 90)
-      (effects (font (size 1.27 1.27)) hide)
-    )
+    (property "Footprint" "Resistor_SMD:R_1206_3216Metric_Pad1.30x1.75mm_HandSolder" (at 26.67 167.132 90)
+      (effects (font (size 1.27 1.27)) hide)
+    )
